File: hardware/sony-scopeman.kicad_pcb (KiCad board)
At the start: 2 copper layers, 53.5 x 101.8 mm, 135 parts, among them J1 EXT_X, J2 COIL_X, J3 EXT_Y, J4 COIL_Y, J5 SPEAKER, J6 USB_C_Receptacle_USB2.0, J7 BLK+CLK, J8 PWR, J9 GND, Q1 PZT3904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

Commit message: Add: Pictures for Instruction
Other:
- board text added: "BLACK PURPLE"
- board text added: "YELLOW BLUE"
- board text removed: "LIGHT BLUE"
Changed lines of the file:
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@@
   (general
     (thickness 1)
-    (drawings 122)
+    (drawings 123)
     (tracks 1000)
     (zones 0)
@@
       (drillshape 0)
       (scaleselection 1)
-      (outputdirectory "gerber_V1.0"))
+      (outputdirectory "gerber_V1.2"))
   )
   (net 0 "")
@@
       (net 18 +4V))
   )
+  (gr_text "BLACK\nPURPLE" (at 123.3 110.1) (layer B.SilkS)
+    (effects (font (size 1 0.7) (thickness 0.15)) (justify mirror))
+  )
   (gr_text "BLACK WHITE" (at 136.8 69.1) (layer B.SilkS)
     (effects (font (size 1 0.7) (thickness 0.15)) (justify mirror))
   )
-  (gr_text "LIGHT BLUE" (at 106.1 83.8) (layer B.SilkS)
+  (gr_text "YELLOW BLUE" (at 111.9 86) (layer B.SilkS)
     (effects (font (size 1 0.7) (thickness 0.15)) (justify mirror))
   )
