File: hardware/sony-scopeman.sch (KiCad schematic (older format))
At the start: 135 parts, among them J1 EXT_X, J2 COIL_X, J3 EXT_Y, J4 COIL_Y, J5 SPEAKER, J6 USB_C_Receptacle_USB2.0, J7 BLK+CLK, J8 PWR, J9 GND, Q1 PZT3904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

Commit message: Add: Pictures for Instruction
Parts:
- R53: value TBD -> 1k
Changed lines of the file:
@@
 P 14850 8700
 F 0 "R53" H 14909 8746 50  0000 L CNN
-F 1 "TBD" H 14909 8655 50  0000 L CNN
+F 1 "1k" H 14909 8655 50  0000 L CNN
 F 2 "Resistor_SMD:R_0603_1608Metric" H 14850 8700 50  0001 C CNN
 F 3 "~" H 14850 8700 50  0001 C CNN
